File: mainboard/rev0/mainboard.sch (EAGLE design)
At the start: 56 parts, among them T1 NPN_BC817,215, T2 NPN_BC817,215, T3 NPN_BC817,215

Commit message: attrs
Parts:
- MAPLE: FARNELL - -> 1593469,1593469
- U$1, U$11: FARNELL 1298480 -> 1095012
Changed lines of the file:
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@@
 <parts>
 <part name="MAPLE" library="rhoban" deviceset="MAPLE_MINI" device="">
-<attribute name="FARNELL" value="-"/>
+<attribute name="FARNELL" value="1593469,1593469"/>
 </part>
 <part name="U$12" library="rhoban" deviceset="NPN" device="_BC817,215">
@@
 </part>
 <part name="U$1" library="to-247_n-channel_igbt" deviceset="TO-247" device="A">
-<attribute name="FARNELL" value="1298480"/>
+<attribute name="FARNELL" value="1095012"/>
 </part>
 <part name="SOLENOID1" library="rhoban" deviceset="CONNEC_1X02" device="BIG">
@@
 </part>
 <part name="U$11" library="to-247_n-channel_igbt" deviceset="TO-247" device="A">
-<attribute name="FARNELL" value="1298480"/>
+<attribute name="FARNELL" value="1095012"/>
 </part>
 <part name="SOLENOID2" library="rhoban" deviceset="CONNEC_1X02" device="BIG">
