File: mainboard/mainboard.sch (EAGLE design)
At the start: 102 parts, among them T1 NPN_BC817,215, T2 NPN_BC817,215, T3 NPN_BC817,215, U1 CD4051BM, X1 JST-XH-10-PIN-LONG-PAD, X2 JST-XH-10-PIN-LONG-PAD, X3 JST-XH-10-PIN-LONG-PAD, X4 JST-XH-10-PIN-LONG-PAD, X5 JST-XH-10-PIN-LONG-PAD

Commit message: Updating mainboard, using brushless drivers [wip]
Parts:
- removed C1, C17, C18, C2, C3, C4, C5, C6: 15pF, rhoban:C_EU_22PF
- removed CA3, CA4, CA5, CA6, CA7: C_EU-100NF, rhoban:C_EU-100NF
- removed ENC1, ENC2, ENC3, ENC4: LS7366RSO14, rhoban:LS7366RSO14
- removed PWM1, PWM2, PWM3, PWM4, PWM5: CONNEC_1X03, rhoban:CONNEC_1X03
- removed R10, R11, R12, R13, R14, R15, R7, R9: 3K, rhoban:RESISTANCE-R0805
- removed R16, R17, R19, R20, R22, R23, R25, R26, R28, R29: 1K, rhoban:RESISTANCE-R0805
- removed R18, R21, R24, R27, R30: 24k, rhoban:RESISTANCE-R0805
- removed U$10, U$6, U$7, U$8, U$9: MAXON380200, rhoban:MAXON380200
- removed U1: CD4051BM, rhoban:CD4051BM
- removed X1, X2, X3, X4, X5: JST-XH-10-PIN-LONG-PAD, Rembrandt Electronics - JST XH Connectors v1-0:JST-XH-10-PIN-LONG-PAD
- removed XTAL1, XTAL2, XTAL3, XTAL4: 40Mhz, rhoban:QUARTZ
- added DRIVER1, DRIVER2, DRIVER3, DRIVER4, DRIVER5: RHOBAN_BL_DRIVER, rhoban:RHOBAN_BL_DRIVER
Connections:
- removed net CS1: ENC1.SS/, R7.2, U1.0
- removed net CS2: ENC2.SS/, R9.2, U1.1
- removed net CS3: ENC3.SS/, R10.2, U1.2
- removed net CS4: ENC4.SS/, R11.2, U1.3
- removed net CS5: COM1.CSN, R12.2, U1.4
- removed net CS6: COM2.CSN, R13.2, U1.5
- removed net CS7: COM3.CSN, R14.2, U1.6
- removed net CS8: R15.2, U1.7
- removed net CSA1: MAPLE.20, U1.A
- removed net CSA2: MAPLE.21, U1.B
- removed net CSA3: MAPLE.22, U1.C
- removed net INDEX: ENC1.INDEX/, ENC2.INDEX/, ENC3.INDEX/, ENC4.INDEX/, MAPLE.26
- removed net M1_A: ENC1.A, X1-9.S
- removed net M1_B: ENC1.B, X1-10.S
- removed net M1_DIR: MAPLE.13, U$6.DIR
- removed net M1_HALL1: U$6.HALL1, X1-6.S
- removed net M1_HALL2: U$6.HALL2, X1-7.S
- removed net M1_HALL3: U$6.HALL3, X1-8.S
- removed net M1_SPEED: MAPLE.3, PWM1.3, U$6.SPEED
- removed net M1_W1: U$6.W1, X1-1.S
- removed net M1_W2: U$6.W2, X1-2.S
- removed net M1_W3: U$6.W3, X1-3.S
- removed net M2_A: ENC2.A, X2-9.S
- removed net M2_B: ENC2.B, X2-10.S
- removed net M2_DIR: MAPLE.14, U$7.DIR
- removed net M2_HALL1: U$7.HALL1, X2-6.S
- removed net M2_HALL2: U$7.HALL2, X2-7.S
- removed net M2_HALL3: U$7.HALL3, X2-8.S
- removed net M2_SPEED: MAPLE.4, PWM2.3, U$7.SPEED
- removed net M2_W1: U$7.W1, X2-1.S
- removed net M2_W2: U$7.W2, X2-2.S
- removed net M2_W3: U$7.W3, X2-3.S
- removed net M3_A: ENC3.A, X3-9.S
- removed net M3_B: ENC3.B, X3-10.S
- removed net M3_DIR: MAPLE.17, U$8.DIR
- removed net M3_HALL1: U$8.HALL1, X3-6.S
- removed net M3_HALL2: U$8.HALL2, X3-7.S
- removed net M3_HALL3: U$8.HALL3, X3-8.S
- removed net M3_SPEED: MAPLE.5, PWM3.3, U$8.SPEED
- removed net M3_W1: U$8.W1, X3-1.S
- removed net M3_W2: U$8.W2, X3-2.S
- removed net M3_W3: U$8.W3, X3-3.S
- removed net M4_A: ENC4.A, X4-9.S
- removed net M4_B: ENC4.B, X4-10.S
- removed net M4_DIR: MAPLE.18, U$9.DIR
- removed net M4_HALL1: U$9.HALL1, X4-6.S
- removed net M4_HALL2: U$9.HALL2, X4-7.S
- removed net M4_HALL3: U$9.HALL3, X4-8.S
- removed net M4_SPEED: MAPLE.8, PWM4.3, U$9.SPEED
- removed net M4_W1: U$9.W1, X4-1.S
- removed net M4_W2: U$9.W2, X4-2.S
- removed net M4_W3: U$9.W3, X4-3.S
- removed net M5_DIR: MAPLE.19, U$10.DIR
- removed net M5_HALL1: U$10.HALL1, X5-6.S
- removed net M5_HALL2: U$10.HALL2, X5-7.S
- removed net M5_HALL3: U$10.HALL3
- removed net M5_SPEED: MAPLE.9, PWM5.3, U$10.SPEED
- removed net M5_W1: U$10.W1, X5-1.S
- removed net M5_W2: U$10.W2, X5-2.S
- removed net M5_W3: U$10.W3, X5-3.S
- removed net MOTORS_EN: U$10.ENABLE, U$6.ENABLE, U$7.ENABLE, U$8.ENABLE, U$9.ENABLE
- removed net MT_HALL3: X5-8.S
- removed net N$10: R16.2, U$6.DIGIN1
- removed net N$12: R17.2, U$6.DIGIN2
- removed net N$13: C1.2, ENC2.FCK0, XTAL2.2
- removed net N$14: C2.2, ENC2.FCKI, XTAL2.1
- removed net N$15: R19.2, U$7.DIGIN1
- removed net N$16: R18.2, U$6.CURRENT
- removed net N$18: R20.2, U$7.DIGIN2
- removed net N$19: C17.2, ENC1.FCK0, XTAL1.2
- removed net N$20: C18.2, ENC1.FCKI, XTAL1.1
- removed net N$21: R21.2, U$7.CURRENT
- removed net N$22: C3.2, ENC3.FCK0, XTAL3.2
- removed net N$23: C4.2, ENC3.FCKI, XTAL3.1
- removed net N$24: R22.2, U$8.DIGIN1
- removed net N$25: R23.2, U$8.DIGIN2
- removed net N$26: R24.2, U$8.CURRENT
- removed net N$27: C5.2, ENC4.FCK0, XTAL4.2
- removed net N$28: C6.2, ENC4.FCKI, XTAL4.1
- removed net N$29: R25.2, U$9.DIGIN1
- removed net N$30: R26.2, U$9.DIGIN2
- removed net N$31: R27.2, U$9.CURRENT
- removed net N$32: R28.2, U$10.DIGIN1
- removed net N$33: R29.2, U$10.DIGIN2
- removed net N$34: R30.2, U$10.CURRENT
- removed net N$8: REG5V.GND
- removed net N$9: REG3.3V.GND
- new net CS_COM_1: COM1.CSN, MAPLE.20
- new net CS_COM_2: COM2.CSN, MAPLE.21
- new net CS_COM_3: COM3.CSN, MAPLE.22
- new net DRIVERS_CS1: DRIVER1.CS, MAPLE.7
- new net DRIVERS_CS2: DRIVER2.CS, MAPLE.26
- new net DRIVERS_CS3: DRIVER3.CS, MAPLE.19
- new net DRIVERS_CS4: DRIVER4.CS, MAPLE.18
- new net DRIVERS_CS5: DRIVER5.CS, MAPLE.17
- new net DRIVERS_MISO: DRIVER1.MISO, DRIVER2.MISO, DRIVER3.MISO, DRIVER4.MISO, DRIVER5.MISO, MAPLE.5
- new net DRIVERS_MOSI: DRIVER1.MOSI, DRIVER2.MOSI, DRIVER3.MOSI, DRIVER4.MOSI, DRIVER5.MOSI, MAPLE.4
- new net DRIVERS_SCK: DRIVER1.SCK, DRIVER2.SCK, DRIVER3.SCK, DRIVER4.SCK, DRIVER5.SCK, MAPLE.6
- new net VMID: DRIVER1.VDRIVER, DRIVER2.VDRIVER, DRIVER3.VDRIVER, DRIVER4.VDRIVER, DRIVER5.VDRIVER, XT1.GND, XT60.V+
- net 3.3: now also DRIVER1.3.3, DRIVER2.3.3, DRIVER3.3.3, DRIVER4.3.3, DRIVER5.3.3; no longer CA3.1, R10.1, R11.1, R12.1, R13.1, R14.1, R15.1, R7.1, R9.1, U1.VDD
- net CAP: now also MAPLE.3; no longer MAPLE.6
- net GND: now also DRIVER1.GND, DRIVER2.GND, DRIVER3.GND, DRIVER4.GND, DRIVER5.GND, REG3.3V.GND, REG5V.GND; no longer C1.1, C17.1, C18.1, C2.1, C3.1, C4.1, C5.1, C6.1, CA3.2, CA4.2, CA5.2, CA6.2, CA7.2, ENC1.VSS, ENC2.VSS, ENC3.VSS, ENC4.VSS, PWM1.1, PWM2.1, PWM3.1, PWM4.1, PWM5.1, R16.1, R18.1, R19.1, R21.1, R22.1, R24.1, R25.1, R27.1, R28.1, R30.1, U$10.GND, U$6.GND, U$7.GND, U$8.GND, U$9.GND, U1.COM_OUT/IN, U1.INH, U1.VEE, U1.VSS, X1-4.S, X2-4.S, X3-4.S, X4-4.S, X5-4.S, XT1.GND
- net MISO: no longer ENC1.MISO, ENC2.MISO, ENC3.MISO, ENC4.MISO
- net MOSI: no longer ENC1.MOSI, ENC2.MOSI, ENC3.MOSI, ENC4.MOSI
- net SCK: no longer ENC1.SCK, ENC2.SCK, ENC3.SCK, ENC4.SCK
- net VCC: now also DRIVER1.VCC, DRIVER2.VCC, DRIVER3.VCC, DRIVER4.VCC, DRIVER5.VCC; no longer CA4.1, CA5.1, CA6.1, CA7.1, ENC1.VDD, ENC2.VDD, ENC3.VDD, ENC4.VDD, R17.1, R20.1, R23.1, R26.1, R29.1, U$10.VCC, U$6.VCC, U$7.VCC, U$8.VCC, U$9.VCC, X1-5.S, X2-5.S, X3-5.S, X4-5.S, X5-5.S
- net VIN: now also DRIVER1.V+, DRIVER2.V+, DRIVER3.V+, DRIVER4.V+, DRIVER5.V+; no longer U$10.VIN, U$6.VIN, U$7.VIN, U$8.VIN, U$9.VIN, XT60.V+
Other:
- note removed: "CS MUX"

Commit message: mainboard
Parts:
- removed CA1, CA2: C_EU-100NF, rhoban:C_EU-100NF
- added C1, C7: 1uF, SparkFun-Passives:CAP0805
- added D1, D2, D3, D4, D5: (no value), SparkFun-DiscreteSemi:DIODESOD
- added R10, R7: 10K, rhoban:RESISTANCE-R0805
- added R11, R9: 1K, rhoban:RESISTANCE-R0805
- BOOST_EN, EMIT, MAPLE, POWERCAP1, POWERCAP2, RECEIVE, SOLENOID1, SOLENOID2, U$13, U$5, XT1, XT60: FARNELL (none) -> -
- COM1, COM2, COM3: FARNELL (none) -> 1668343
- DRIVER1, DRIVER2, DRIVER3, DRIVER4, DRIVER5: FARNELL (none) -> 1593459,1593459,1593463
- R1, R31, R4: FARNELL (none) -> 2446904
- R2, R3, R32, R33, R36, R8: FARNELL (none) -> 2446965
- R34: FARNELL (none) -> 2129375
- R35, R6: FARNELL (none) -> 2447553
- R5: value 110 -> 62; FARNELL (none) -> 2138819
- REG3.3V: FARNELL (none) -> 1696319
- REG5V: FARNELL (none) -> 1696320
- T1, T2, T3, U$12, U$15: FARNELL (none) -> 1081223
- U$1, U$11: FARNELL (none) -> 1298480
- U$2: FARNELL (none) -> 1593463
- U$3, U$4: FARNELL (none) -> 9696946
Connections:
- new net BAT1: MAPLE.8, R7.1, R9.2
- new net BAT2: MAPLE.9, R10.1, R11.2
- new net N$10: D4.C, DRIVER5.VDRIVER
- new net N$12: D2.C, DRIVER3.VDRIVER
- new net N$13: D1.C, DRIVER2.VDRIVER
- new net N$8: D5.C, DRIVER1.VDRIVER
- new net N$9: D3.C, DRIVER4.VDRIVER
- net 3.3: now also C7.2; no longer CA1.1
- net GND: now also C1.1, C7.1, R11.1, R9.1; no longer CA1.2, CA2.2
- net VBOOST: now also R10.2, R7.2
- net VCC: now also C1.2; no longer CA2.1
- net VMID: now also D1.A, D2.A, D3.A, D4.A, D5.A; no longer DRIVER1.VDRIVER, DRIVER2.VDRIVER, DRIVER3.VDRIVER, DRIVER4.VDRIVER, DRIVER5.VDRIVER
Other:
- moved on the sheet: POWERCAP1, POWERCAP2, R34, R35, SOLENOID1, U$4

Commit message: mainboard
Connections:
- new net COM_CE: COM1.CE, COM2.CE, COM3.CE, MAPLE.13
- net 3.3: no longer COM1.CE, COM2.CE, COM3.CE
- net VBOOST: no longer R10.2, R7.2
- net VIN: now also R10.2
- net VMID: now also R7.2

Commit message: attrs
Parts:
- MAPLE: FARNELL - -> 1593469,1593469
- U$1, U$11: FARNELL 1298480 -> 1095012
Changed lines of the file:
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@@
 <parts>
 <part name="MAPLE" library="rhoban" deviceset="MAPLE_MINI" device="">
-<attribute name="FARNELL" value="-"/>
+<attribute name="FARNELL" value="1593469,1593469"/>
 </part>
 <part name="U$12" library="rhoban" deviceset="NPN" device="_BC817,215">
@@
 </part>
 <part name="U$1" library="to-247_n-channel_igbt" deviceset="TO-247" device="A">
-<attribute name="FARNELL" value="1298480"/>
+<attribute name="FARNELL" value="1095012"/>
 </part>
 <part name="SOLENOID1" library="rhoban" deviceset="CONNEC_1X02" device="BIG">
@@
 </part>
 <part name="U$11" library="to-247_n-channel_igbt" deviceset="TO-247" device="A">
-<attribute name="FARNELL" value="1298480"/>
+<attribute name="FARNELL" value="1095012"/>
 </part>
 <part name="SOLENOID2" library="rhoban" deviceset="CONNEC_1X02" device="BIG">

Commit message: Mainboard rev1 wip
Parts:
- removed BOOST_EN: CONNEC_1X01, rhoban:CONNEC_1X01
- removed POWERCAP1, POWERCAP2, SOLENOID1, SOLENOID2: CONNEC_1X02BIG, rhoban:CONNEC_1X02BIG
- removed R31, R9: 1K, rhoban:RESISTANCE-R0805
- removed R32, R33, R36: 3K, rhoban:RESISTANCE-R0805
- removed R34: 2M, rhoban:RESISTANCE-R0805
- removed R35: 10K, rhoban:RESISTANCE-R0805
- removed T1, T3, U$15: NPN_BC817,215, rhoban:NPN_BC817,215
- removed XT1: CONNEC_ALIM, rhoban:CONNEC_ALIM
- added C2: 1uF, SparkFun-Passives:CAP0805
- added REG3.3V1: REG_5V, rhoban:REG_5V
- added U$10: DRV5023FAEDBZRQ1, rhoban:DRV5023FAEDBZRQ1
- added U$6: 47uF, rhoban:CPOL_EUPANASONIC_D
- added U$7, U$8, U$9: (no value), rhoban:CPOL_EUPANASONIC_D8
- added X1: JST-XH-06-PIN-LONG-PAD, Rembrandt Electronics - JST XH Connectors v1-0:JST-XH-06-PIN-LONG-PAD
- R1: value 1K -> 10K; FARNELL 2446904 -> 2447553
- R2, R3: value 3K -> 10K; FARNELL 2446965 -> 2447553
- U$1, U$11: value TO-247A -> DRV5023FAEDBZRQ1; device to-247_n-channel_igbt:TO-247A -> rhoban:DRV5023FAEDBZRQ1; FARNELL 1095012 -> (none)
- U$5: value BOOSTER -> DRV5023FAEDBZRQ1; device rhoban:BOOSTER -> rhoban:DRV5023FAEDBZRQ1; FARNELL - -> (none)
Connections:
- net BAT2 renamed BAT
- removed net BAT1: MAPLE.8, R7.1, R9.2
- removed net N$1: R1.2, T1.B
- removed net N$17: R31.2, T3.B
- removed net N$2: SOLENOID1.2, U$1.C
- removed net N$35: R33.1, T3.C, U$11.G
- removed net N$36: SOLENOID2.2, U$11.C
- removed net N$37: BOOST_EN.1, U$15.C
- removed net N$38: R36.1, U$15.B
- removed net N$4: R3.1, T1.C, U$1.G
- removed net VBOOST: POWERCAP1.2, POWERCAP2.2, R34.2, SOLENOID1.1, SOLENOID2.1, U$5.OUT+
- removed net VMID: D1.A, D2.A, D3.A, D4.A, D5.A, R7.2, XT1.GND, XT60.V+
- new net 12V: C2.2, D1.A, D2.A, D3.A, D4.A, D5.A, REG3.3V1.OUT, U$6.+
- new net HALL1: MAPLE.14, R1.1, U$1.OUT
- new net HALL2: MAPLE.8, R2.1, U$5.OUT
- new net HALL3: MAPLE.2, R3.1, U$10.OUT
- new net HALL4: MAPLE.31, R7.1, U$11.OUT
- net 3.3: now also R1.2, R3.2, R7.2, U$1.VCC, U$10.VCC, U$11.VCC, U$5.VCC, U$7.+, U$8.+, U$9.+; no longer R32.2
- net BOOST_EN: now also X1-3.S; no longer R36.2
- net CAP: now also X1-6.S; no longer R34.1, R35.2
- net GND: now also C2.1, REG3.3V1.GND, U$1.GND, U$10.GND, U$11.GND, U$5.GND, U$6.-, U$7.-, U$8.-, U$9.-, X1-1.S; no longer POWERCAP1.1, POWERCAP2.1, R35.1, R9.1, T1.E, T3.E, U$1.E, U$11.E, U$15.E, U$5.IN-, U$5.OUT-
- net KICK1: now also X1-4.S; no longer R1.1, R2.1
- net KICK2: now also X1-5.S; no longer R31.1, R32.1
- net VIN: now also REG3.3V1.IN, X1-2.S, XT60.V+; no longer R3.2, R33.2, U$5.IN+, XT1.V+
Other:
- note added: "HALL"

Commit message: Updating designs
Connections:
- net DRIVERS_CS2: now also MAPLE.1; no longer MAPLE.26
- net IRQ3: now also MAPLE.0; no longer MAPLE.25
- net KICK1: now also MAPLE.25; no longer MAPLE.0
- net KICK2: now also MAPLE.26; no longer MAPLE.1

Commit message: mainboard updates
Parts:
- added U$15: SRB22A2FBBNN, rhoban:SRB22A2FBBNN
Connections:
- new net VIN_BAT: U$15.P$2, XT60.V+
- net VIN: now also U$15.P$1; no longer XT60.V+
Changed lines of the file:
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@@
 <attribute name="FARNELL" value="2447553"/>
 </part>
+<part name="U$15" library="rhoban" deviceset="SRB22A2FBBNN" device=""/>
 </parts>
 <sheets>
@@
 <attribute name="FARNELL" x="-45.72" y="-60.96" size="1.778" layer="96" rot="R90" display="off"/>
 </instance>
+<instance part="U$15" gate="G$1" x="-58.42" y="-15.24"/>
 </instances>
 <busses>
@@
 <pinref part="R11" gate="G$1" pin="1"/>
 <wire x1="-45.72" y1="-71.12" x2="-45.72" y2="-66.04" width="0.1524" layer="91"/>
-<label x="-45.72" y="-71.12" size="1.27" layer="95" rot="R270" xref="yes"/>
+<label x="-45.72" y="-71.12" size="1.27" layer="95" xref="yes"/>
 </segment>
 </net>
@@
 </segment>
 <segment>
-<pinref part="XT60" gate="G$1" pin="V+"/>
-<wire x1="-48.26" y1="5.08" x2="-55.88" y2="5.08" width="0.1524" layer="91"/>
-<label x="-55.88" y="5.08" size="1.27" layer="95" rot="R180" xref="yes"/>
-</segment>
-<segment>
 <pinref part="R10" gate="G$1" pin="2"/>
 <wire x1="-45.72" y1="-40.64" x2="-45.72" y2="-38.1" width="0.1524" layer="91"/>
-<label x="-45.72" y="-38.1" size="1.27" layer="95" rot="R90" xref="yes"/>
+<label x="-45.72" y="-38.1" size="1.27" layer="95" xref="yes"/>
+</segment>
+<segment>
+<pinref part="U$15" gate="G$1" pin="P$1"/>
+<wire x1="-60.96" y1="-15.24" x2="-66.04" y2="-15.24" width="0.1524" layer="91"/>
+<label x="-66.04" y="-15.24" size="1.27" layer="95" rot="R180" xref="yes"/>
 </segment>
 </net>
@@
 </segment>
 </net>
+<net name="VIN_BAT" class="2">
+<segment>
+<pinref part="XT60" gate="G$1" pin="V+"/>
+<wire x1="-48.26" y1="5.08" x2="-55.88" y2="5.08" width="0.1524" layer="91"/>
+<label x="-55.88" y="5.08" size="1.27" layer="95" rot="R180" xref="yes"/>
+</segment>
+<segment>
+<pinref part="U$15" gate="G$1" pin="P$2"/>
+<wire x1="-33.02" y1="-15.24" x2="-27.94" y2="-15.24" width="0.1524" layer="91"/>
+<label x="-27.94" y="-15.24" size="1.27" layer="95" xref="yes"/>
+</segment>
+</net>

Commit message: Update mainboard
Parts:
- U$15: FARNELL (none) -> 1383947
Changed lines of the file:
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@@
 <attribute name="FARNELL" value="2447553"/>
 </part>
-<part name="U$15" library="rhoban" deviceset="SRB22A2FBBNN" device=""/>
+<part name="U$15" library="rhoban" deviceset="SRB22A2FBBNN" device="">
+<attribute name="FARNELL" value="1383947"/>
+</part>
 </parts>
 <sheets>
@@
 <attribute name="FARNELL" x="-45.72" y="-60.96" size="1.778" layer="96" rot="R90" display="off"/>
 </instance>
-<instance part="U$15" gate="G$1" x="-58.42" y="-15.24"/>
+<instance part="U$15" gate="G$1" x="-58.42" y="-15.24">
+<attribute name="FARNELL" x="-58.42" y="-15.24" size="1.778" layer="96" display="off"/>
+</instance>
 </instances>
 <busses>
