File: kicker/kicker.brd (EAGLE design)
At the start: 59.7 x 56.3 mm, 35 parts, among them Q1 BSS123, Q2 BSS123, X2 JST-XH-07-PIN-LONG-PAD

Commit message: Values
Parts:
- C1, C2: value (none) -> 1uF
- D1: value (none) -> 3.9V
- D5: value (none) -> 12V
Changed lines of the file:
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@@
 <layer number="25" name="tNames" color="7" fill="1" visible="yes" active="yes"/>
 <layer number="26" name="bNames" color="7" fill="1" visible="yes" active="yes"/>
-<layer number="27" name="tValues" color="7" fill="1" visible="no" active="yes"/>
-<layer number="28" name="bValues" color="7" fill="1" visible="no" active="yes"/>
-<layer number="29" name="tStop" color="7" fill="3" visible="no" active="yes"/>
-<layer number="30" name="bStop" color="7" fill="6" visible="no" active="yes"/>
-<layer number="31" name="tCream" color="7" fill="4" visible="no" active="yes"/>
-<layer number="32" name="bCream" color="7" fill="5" visible="no" active="yes"/>
-<layer number="33" name="tFinish" color="6" fill="3" visible="no" active="yes"/>
-<layer number="34" name="bFinish" color="6" fill="6" visible="no" active="yes"/>
-<layer number="35" name="tGlue" color="7" fill="4" visible="no" active="yes"/>
-<layer number="36" name="bGlue" color="7" fill="5" visible="no" active="yes"/>
+<layer number="27" name="tValues" color="7" fill="1" visible="yes" active="yes"/>
+<layer number="28" name="bValues" color="7" fill="1" visible="yes" active="yes"/>
+<layer number="29" name="tStop" color="7" fill="3" visible="yes" active="yes"/>
+<layer number="30" name="bStop" color="7" fill="6" visible="yes" active="yes"/>
+<layer number="31" name="tCream" color="7" fill="4" visible="yes" active="yes"/>
+<layer number="32" name="bCream" color="7" fill="5" visible="yes" active="yes"/>
+<layer number="33" name="tFinish" color="6" fill="3" visible="yes" active="yes"/>
+<layer number="34" name="bFinish" color="6" fill="6" visible="yes" active="yes"/>
+<layer number="35" name="tGlue" color="7" fill="4" visible="yes" active="yes"/>
+<layer number="36" name="bGlue" color="7" fill="5" visible="yes" active="yes"/>
 <layer number="37" name="tTest" color="7" fill="1" visible="yes" active="yes"/>
 <layer number="38" name="bTest" color="7" fill="1" visible="yes" active="yes"/>
@@
 <layer number="42" name="bRestrict" color="1" fill="10" visible="yes" active="yes"/>
 <layer number="43" name="vRestrict" color="2" fill="10" visible="yes" active="yes"/>
-<layer number="44" name="Drills" color="7" fill="1" visible="no" active="yes"/>
-<layer number="45" name="Holes" color="7" fill="1" visible="no" active="yes"/>
+<layer number="44" name="Drills" color="7" fill="1" visible="yes" active="yes"/>
+<layer number="45" name="Holes" color="7" fill="1" visible="yes" active="yes"/>
 <layer number="46" name="Milling" color="3" fill="1" visible="yes" active="yes"/>
-<layer number="47" name="Measures" color="7" fill="1" visible="no" active="yes"/>
+<layer number="47" name="Measures" color="7" fill="1" visible="yes" active="yes"/>
 <layer number="48" name="Document" color="7" fill="1" visible="yes" active="yes"/>
-<layer number="49" name="Reference" color="7" fill="1" visible="no" active="yes"/>
+<layer number="49" name="Reference" color="7" fill="1" visible="yes" active="yes"/>
 <layer number="50" name="dxf" color="7" fill="1" visible="no" active="no"/>
-<layer number="51" name="tDocu" color="7" fill="1" visible="no" active="yes"/>
-<layer number="52" name="bDocu" color="7" fill="1" visible="no" active="yes"/>
+<layer number="51" name="tDocu" color="7" fill="1" visible="yes" active="yes"/>
+<layer number="52" name="bDocu" color="7" fill="1" visible="yes" active="yes"/>
 <layer number="53" name="tGND_GNDA" color="7" fill="9" visible="no" active="no"/>
 <layer number="54" name="bGND_GNDA" color="1" fill="9" visible="no" active="no"/>
@@
 <attribute name="VALUE" x="43.18" y="24.003" size="1.27" layer="27" ratio="10" rot="R180"/>
 <attribute name="NAME" x="43.434" y="20.447" size="1.27" layer="25" ratio="10" rot="R180"/>
+<attribute name="FARNELL" value="9551735" x="40.64" y="21.844" size="1.778" layer="27" rot="R180" display="off"/>
 </element>
 <element name="D3" library="diode" package="C4111-15" value="1N6267A" x="18.542" y="21.844" smashed="yes" rot="R180">
 <attribute name="VALUE" x="21.082" y="24.003" size="1.27" layer="27" ratio="10" rot="R180"/>
 <attribute name="NAME" x="20.066" y="20.701" size="1.27" layer="25" ratio="10" rot="R180"/>
-</element>
-<element name="C1" library="rcl" package="C0805" value="" x="26.924" y="41.91" smashed="yes" rot="MR180">
+<attribute name="FARNELL" value="9551735" x="18.542" y="21.844" size="1.778" layer="27" rot="R180" display="off"/>
+</element>
+<element name="C1" library="rcl" package="C0805" value="1uF" x="26.924" y="41.91" smashed="yes" rot="MR180">
 <attribute name="NAME" x="25.908" y="44.45" size="1.27" layer="26" rot="MR180"/>
 <attribute name="VALUE" x="25.654" y="44.45" size="1.27" layer="28" rot="MR180"/>
 </element>
-<element name="C2" library="rcl" package="C0805" value="" x="49.022" y="42.418" smashed="yes" rot="MR180">
+<element name="C2" library="rcl" package="C0805" value="1uF" x="49.022" y="42.418" smashed="yes" rot="MR180">
 <attribute name="NAME" x="47.498" y="44.958" size="1.27" layer="26" rot="MR180"/>
 <attribute name="VALUE" x="47.752" y="44.958" size="1.27" layer="28" rot="MR180"/>
@@
 <attribute name="VALUE" x="20.574" y="2.794" size="0.4064" layer="28" rot="MR180"/>
 </element>
-<element name="D5" library="diode" package="SOD80C" value="" x="15.494" y="1.524" smashed="yes" rot="MR0">
+<element name="D5" library="diode" package="SOD80C" value="12V" x="15.494" y="1.524" smashed="yes" rot="MR0">
 <attribute name="NAME" x="16.002" y="-1.143" size="1.27" layer="26" rot="MR0"/>
 <attribute name="VALUE" x="17.018" y="-0.889" size="1.27" layer="28" rot="MR0"/>
-</element>
-<element name="D1" library="diode" package="SOD80C" value="" x="49.784" y="8.382" smashed="yes" rot="R270">
+<attribute name="FARNELL" value="2319144" x="15.494" y="1.524" size="1.778" layer="28" rot="MR0" display="off"/>
+</element>
+<element name="D1" library="diode" package="SOD80C" value="3.9V" x="49.784" y="8.382" smashed="yes" rot="R270">
 <attribute name="NAME" x="47.117" y="9.398" size="1.27" layer="25" rot="R270"/>
 <attribute name="VALUE" x="47.371" y="9.906" size="1.27" layer="27" rot="R270"/>
+<attribute name="FARNELL" value="1097198" x="49.784" y="8.382" size="1.778" layer="27" rot="R270" display="off"/>
 </element>
 </elements>

Commit message: Passive values
Parts:
- R1, R2, R4, R7: value 3K -> 470
- R10, R11: value 10K -> 100K
- R8: value 3K -> 100K
Changed lines of the file:
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@@
 <attribute name="NAME" x="44.196" y="41.3385" size="1.27" layer="26" ratio="10" rot="MR0"/>
 </element>
-<element name="R1" library="rhoban" package="R0805" value="3K" x="49.022" y="36.83" smashed="yes" rot="MR180">
+<element name="R1" library="rhoban" package="R0805" value="470" x="49.022" y="36.83" smashed="yes" rot="MR180">
 <attribute name="FARNELL" value="2446965" x="49.022" y="36.83" size="1.778" layer="28" rot="MR180" display="off"/>
 <attribute name="VALUE" x="49.022" y="38.1" size="0.4064" layer="28" rot="MR180"/>
@@
 <attribute name="NAME" x="22.352" y="40.5765" size="1.27" layer="26" ratio="10" rot="MR0"/>
 </element>
-<element name="R2" library="rhoban" package="R0805" value="3K" x="26.924" y="36.83" smashed="yes" rot="MR180">
+<element name="R2" library="rhoban" package="R0805" value="470" x="26.924" y="36.83" smashed="yes" rot="MR180">
 <attribute name="FARNELL" value="2446965" x="17.78" y="45.974" size="1.778" layer="28" rot="MR180" display="off"/>
 <attribute name="VALUE" x="26.924" y="38.1" size="0.4064" layer="28" rot="MR180"/>
@@
 <attribute name="VALUE" x="52.07" y="17.272" size="0.4064" layer="27" rot="R90"/>
 </element>
-<element name="R4" library="rhoban" package="R0805" value="3K" x="26.924" y="39.37" smashed="yes" rot="MR180">
+<element name="R4" library="rhoban" package="R0805" value="470" x="26.924" y="39.37" smashed="yes" rot="MR180">
 <attribute name="FARNELL" value="2446965" x="26.924" y="39.37" size="1.778" layer="28" rot="MR180" display="off"/>
 <attribute name="VALUE" x="26.924" y="40.64" size="0.4064" layer="28" rot="MR180"/>
 </element>
-<element name="R7" library="rhoban" package="R0805" value="3K" x="49.022" y="39.878" smashed="yes" rot="MR180">
+<element name="R7" library="rhoban" package="R0805" value="470" x="49.022" y="39.878" smashed="yes" rot="MR180">
 <attribute name="FARNELL" value="2446965" x="49.022" y="39.878" size="1.778" layer="28" rot="MR180" display="off"/>
 <attribute name="VALUE" x="49.022" y="41.148" size="0.4064" layer="28" rot="MR180"/>
@@
 <attribute name="VALUE" x="47.752" y="44.958" size="1.27" layer="28" rot="MR180"/>
 </element>
-<element name="R8" library="rhoban" package="R0805" value="3K" x="11.684" y="41.656" smashed="yes" rot="MR0">
+<element name="R8" library="rhoban" package="R0805" value="100K" x="11.684" y="41.656" smashed="yes" rot="MR0">
 <attribute name="FARNELL" value="2446965" x="11.684" y="41.656" size="1.778" layer="28" rot="MR0" display="off"/>
 <attribute name="VALUE" x="11.684" y="40.386" size="0.4064" layer="28" rot="MR0"/>
@@
 <attribute name="VALUE" x="16.764" y="6.858" size="0.4064" layer="28" rot="MR180"/>
 </element>
-<element name="R10" library="rhoban" package="R0805" value="10K" x="25.654" y="1.524" smashed="yes" rot="MR180">
+<element name="R10" library="rhoban" package="R0805" value="100K" x="25.654" y="1.524" smashed="yes" rot="MR180">
 <attribute name="FARNELL" value="2447553" x="25.654" y="1.524" size="1.778" layer="28" rot="MR180" display="off"/>
 <attribute name="VALUE" x="25.654" y="2.794" size="0.4064" layer="28" rot="MR180"/>
 </element>
-<element name="R11" library="rhoban" package="R0805" value="10K" x="20.574" y="1.524" smashed="yes" rot="MR180">
+<element name="R11" library="rhoban" package="R0805" value="100K" x="20.574" y="1.524" smashed="yes" rot="MR180">
 <attribute name="FARNELL" value="2447553" x="20.574" y="1.524" size="1.778" layer="28" rot="MR180" display="off"/>
 <attribute name="VALUE" x="20.574" y="2.794" size="0.4064" layer="28" rot="MR180"/>
