File: kicker/rev0/kicker.brd (EAGLE design)
At the start: 59.7 x 56.3 mm, 28 parts, among them T1 NPN_BC817,215, T2 NPN_BC817,215, T3 NPN_BC817,215, T4 NPN_BC817,215, X1 JST-XH-06-PIN-LONG-PAD

Commit message: rearranging rev0 board for 2 big moses
Parts:
- removed U$2, U$3: (no value), SparkFun-Hardware:STAND-OFF
- moved R8 46.5 mm to (20.6, 48.0), flipped to the bottom, turned to 0 degrees
- moved R33 44.3 mm to (15.2, 43.2), flipped to the bottom, turned to 90 degrees
- moved R6 39.9 mm to (13.0, 37.6), flipped to the bottom, turned to 90 degrees
- moved U$4 38.3 mm to (26.2, 45.5), flipped to the bottom
- moved T3 38.1 mm to (16.5, 38.6), flipped to the bottom, turned to 270 degrees
- moved R2 37.9 mm to (10.4, 37.6), flipped to the bottom, turned to 270 degrees
- moved T4 37.6 mm to (31.2, 44.2), flipped to the bottom, turned to 0 degrees
- moved R7 36.1 mm to (31.2, 48.0), flipped to the bottom, turned to 180 degrees
- moved R34 35.8 mm to (52.3, 44.2), flipped to the bottom, turned to 90 degrees
- moved T2 35.2 mm to (20.6, 44.5), flipped to the bottom, turned to 0 degrees
- moved R35 30.8 mm to (52.3, 39.6), flipped to the bottom, turned to 90 degrees
- moved R36 28.7 mm to (9.91, 42.7), flipped to the bottom, turned to 270 degrees
- moved BOOST_EN 28.7 mm to (2.54, 42.7)
- moved U$15 28.7 mm to (6.35, 42.7), flipped to the bottom, turned to 270 degrees
- moved R32 26.3 mm to (31.8, 37.8), flipped to the bottom, turned to 270 degrees
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Routing:
- net KICK2: track 16.7 -> 84.2 mm, vias 1 -> 2
- net N$8: track 63.1 -> 13.1 mm, vias 0 -> 1
- net KICK1: track 17.7 -> 59.5 mm
- net KICK_TR1: track 16.8 -> 54.4 mm, vias 2 -> 4
- net KICK_TR2: track 20.7 -> 57.7 mm
- net GND: track 165.3 -> 201.3 mm, vias 13 -> 5
- net CAP: track 16.4 -> 44.7 mm, vias 0 -> 1
- net BOOST_EN: track 97.6 -> 70.4 mm, vias 0 -> 1
- net VBOOST: track 43.0 -> 68.0 mm, vias 2 -> 1
- net VIN: track 137.1 -> 161.7 mm
- net KICK2R: track 13.7 -> 32.5 mm, vias 3 -> 4
- net N$7: track 25.4 -> 12.9 mm, vias 2 -> 1
- net N$2: track 11.6 -> 18.8 mm
- net KICK1R: track 10.6 -> 13.2 mm, vias 2 -> 0
- net N$36: track 11.4 -> 9.40 mm
