File: brushless/rev2/brushless.sch (EAGLE design)
At the start: 72 parts, among them Q1 BUK7Y12-40E, Q2 BUK7Y12-40E, Q3 BUK7Y12-40E, Q4 BUK7Y12-40E, Q5 BUK7Y12-40E, Q6 BUK7Y12-40E, X2 MOTOR

Commit message: Passive values
Parts:
- C11: value 1000pF -> 1uF
- C13: value 1000pF -> 100nF
Changed lines of the file:
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@@
 <attribute name="FARNELL" value="2496935"/>
 </part>
-<part name="C11" library="SparkFun-Passives" deviceset="CAP" device="0805" value="1000pF">
+<part name="C11" library="SparkFun-Passives" deviceset="CAP" device="0805" value="1uF">
 <attribute name="FARNELL" value="2496935"/>
 </part>
-<part name="C13" library="SparkFun-Passives" deviceset="CAP" device="0805" value="1000pF">
+<part name="C13" library="SparkFun-Passives" deviceset="CAP" device="0805" value="100nF">
 <attribute name="FARNELL" value="2496935"/>
 </part>
