File: brushless/rev2/brushless.sch (EAGLE design)
At the start: 72 parts, among them Q1 BUK7Y12-40E, Q2 BUK7Y12-40E, Q3 BUK7Y12-40E, Q4 BUK7Y12-40E, Q5 BUK7Y12-40E, Q6 BUK7Y12-40E, X2 MOTOR

Commit message: Bootstrap values
Parts:
- C1, C2, C3: value 10µF -> 1µF
Changed lines of the file:
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@@
 <?xml version="1.0" encoding="utf-8"?>
 <!DOCTYPE eagle SYSTEM "eagle.dtd">
-<eagle version="6.1">
+<eagle version="8.7.0">
 <drawing>
 <settings>
 <setting alwaysvectorfont="no"/>
+<setting keepoldvectorfont="yes"/>
 <setting verticaltext="up"/>
 </settings>
@@
 <attribute name="FARNELL" value="8638730"/>
 </part>
-<part name="C1" library="SparkFun-Capacitors" deviceset="0.33UF/330NF" device="-0805-50V-10%" value="10µF">
+<part name="C1" library="SparkFun-Capacitors" deviceset="0.33UF/330NF" device="-0805-50V-10%" value="1µF">
 <attribute name="FARNELL" value="2528772"/>
 </part>
@@
 <attribute name="FARNELL" value="8638730"/>
 </part>
-<part name="C2" library="SparkFun-Capacitors" deviceset="0.33UF/330NF" device="-0805-50V-10%" value="10µF">
+<part name="C2" library="SparkFun-Capacitors" deviceset="0.33UF/330NF" device="-0805-50V-10%" value="1µF">
 <attribute name="FARNELL" value="2528772"/>
 </part>
@@
 <attribute name="FARNELL" value="8638730"/>
 </part>
-<part name="C3" library="SparkFun-Capacitors" deviceset="0.33UF/330NF" device="-0805-50V-10%" value="10µF">
+<part name="C3" library="SparkFun-Capacitors" deviceset="0.33UF/330NF" device="-0805-50V-10%" value="1µF">
 <attribute name="FARNELL" value="2528772"/>
 </part>

Commit message: Passive values
Parts:
- C11: value 1000pF -> 1uF
- C13, C9: value 1000pF -> 100nF
Changed lines of the file:
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@@
 <?xml version="1.0" encoding="utf-8"?>
 <!DOCTYPE eagle SYSTEM "eagle.dtd">
-<eagle version="8.7.0">
+<eagle version="6.1">
 <drawing>
 <settings>
 <setting alwaysvectorfont="no"/>
-<setting keepoldvectorfont="yes"/>
 <setting verticaltext="up"/>
 </settings>
@@
 <part name="AGND19" library="supply1" deviceset="AGND" device=""/>
 <part name="AGND20" library="supply1" deviceset="AGND" device=""/>
-<part name="C9" library="SparkFun-Passives" deviceset="CAP" device="0805" value="1000pF">
+<part name="C9" library="SparkFun-Passives" deviceset="CAP" device="0805" value="100nF">
 <attribute name="FARNELL" value="2496935"/>
 </part>
-<part name="C11" library="SparkFun-Passives" deviceset="CAP" device="0805" value="1000pF">
+<part name="C11" library="SparkFun-Passives" deviceset="CAP" device="0805" value="1uF">
 <attribute name="FARNELL" value="2496935"/>
 </part>
-<part name="C13" library="SparkFun-Passives" deviceset="CAP" device="0805" value="1000pF">
+<part name="C13" library="SparkFun-Passives" deviceset="CAP" device="0805" value="100nF">
 <attribute name="FARNELL" value="2496935"/>
 </part>

Commit message: Improving values indications
Parts:
- D1, D10, D11, D7, D8, D9: value (none) -> Signal; FARNELL 8737843RL -> 1843678RL
- D12, D2, D3, D5, D6: value (none) -> Schottky; FARNELL 8737843RL -> 2760406
Changed lines of the file:
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@@
 <attribute name="FARNELL" value="1870964"/>
 </part>
-<part name="D5" library="SparkFun-DiscreteSemi" deviceset="DIODE" device="SOD">
-<attribute name="FARNELL" value="8737843RL"/>
+<part name="D5" library="SparkFun-DiscreteSemi" deviceset="DIODE" device="SOD" value="Schottky">
+<attribute name="FARNELL" value="2760406"/>
 </part>
 <part name="JP1" library="SparkFun-Jumpers" deviceset="JUMPER-SMT_2_NC_PASTE" device="_NO-SILK">
@@
 </part>
 <part name="3.3/4.5D3" library="supply1" deviceset="+3V3" device=""/>
-<part name="D6" library="SparkFun-DiscreteSemi" deviceset="DIODE" device="SOD">
-<attribute name="FARNELL" value="8737843RL"/>
+<part name="D6" library="SparkFun-DiscreteSemi" deviceset="DIODE" device="SOD" value="Schottky">
+<attribute name="FARNELL" value="2760406"/>
 </part>
-<part name="D1" library="SparkFun-DiscreteSemi" deviceset="DIODE" device="SOD">
-<attribute name="FARNELL" value="8737843RL"/>
+<part name="D1" library="SparkFun-DiscreteSemi" deviceset="DIODE" device="SOD" value="Signal">
+<attribute name="FARNELL" value="1843678RL"/>
 </part>
-<part name="D2" library="SparkFun-DiscreteSemi" deviceset="DIODE" device="SOD">
-<attribute name="FARNELL" value="8737843RL"/>
+<part name="D2" library="SparkFun-DiscreteSemi" deviceset="DIODE" device="SOD" value="Schottky">
+<attribute name="FARNELL" value="2760406"/>
 </part>
-<part name="D7" library="SparkFun-DiscreteSemi" deviceset="DIODE" device="SOD">
-<attribute name="FARNELL" value="8737843RL"/>
+<part name="D7" library="SparkFun-DiscreteSemi" deviceset="DIODE" device="SOD" value="Signal">
+<attribute name="FARNELL" value="1843678RL"/>
 </part>
-<part name="D8" library="SparkFun-DiscreteSemi" deviceset="DIODE" device="SOD">
-<attribute name="FARNELL" value="8737843RL"/>
+<part name="D8" library="SparkFun-DiscreteSemi" deviceset="DIODE" device="SOD" value="Signal">
+<attribute name="FARNELL" value="1843678RL"/>
 </part>
-<part name="D9" library="SparkFun-DiscreteSemi" deviceset="DIODE" device="SOD">
-<attribute name="FARNELL" value="8737843RL"/>
+<part name="D9" library="SparkFun-DiscreteSemi" deviceset="DIODE" device="SOD" value="Signal">
+<attribute name="FARNELL" value="1843678RL"/>
 </part>
-<part name="D3" library="SparkFun-DiscreteSemi" deviceset="DIODE" device="SOD">
-<attribute name="FARNELL" value="8737843RL"/>
+<part name="D3" library="SparkFun-DiscreteSemi" deviceset="DIODE" device="SOD" value="Schottky">
+<attribute name="FARNELL" value="2760406"/>
 </part>
-<part name="D10" library="SparkFun-DiscreteSemi" deviceset="DIODE" device="SOD">
-<attribute name="FARNELL" value="8737843RL"/>
+<part name="D10" library="SparkFun-DiscreteSemi" deviceset="DIODE" device="SOD" value="Signal">
+<attribute name="FARNELL" value="1843678RL"/>
 </part>
-<part name="D11" library="SparkFun-DiscreteSemi" deviceset="DIODE" device="SOD">
-<attribute name="FARNELL" value="8737843RL"/>
+<part name="D11" library="SparkFun-DiscreteSemi" deviceset="DIODE" device="SOD" value="Signal">
+<attribute name="FARNELL" value="1843678RL"/>
 </part>
-<part name="D12" library="SparkFun-DiscreteSemi" deviceset="DIODE" device="SOD">
-<attribute name="FARNELL" value="8737843RL"/>
+<part name="D12" library="SparkFun-DiscreteSemi" deviceset="DIODE" device="SOD" value="Schottky">
+<attribute name="FARNELL" value="2760406"/>
 </part>
 <part name="R7" library="SparkFun-Resistors" deviceset="RESISTOR" device="0805" value="10">

Commit message: Farnell BOM attributes
Parts:
- C1, C2, C3: FARNELL 2528772 -> 2496946
- C11: FARNELL 2496935 -> 2496946
- C13, C9: FARNELL 2496935 -> 1759143RL
- C4: FARNELL 2496935 -> 2392334
- D12, D2, D3, D5, D6: FARNELL 2760406 -> 8734593
- DRV1, DRV2, DRV3: FARNELL 8638730 -> 8638756
- R1, R10, R11, R12, R2, R3, R4, R5, R6, R7, R8, R9: FARNELL 2446904 -> 2498048
Changed lines of the file:
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@@
 </part>
 <part name="DRV1" library="rhoban" deviceset="OPEN-BLDC_IR2101" device="">
-<attribute name="FARNELL" value="8638730"/>
+<attribute name="FARNELL" value="8638756"/>
 </part>
 <part name="C1" library="SparkFun-Capacitors" deviceset="0.33UF/330NF" device="-0805-50V-10%" value="1µF">
-<attribute name="FARNELL" value="2528772"/>
+<attribute name="FARNELL" value="2496946"/>
 </part>
 <part name="DRV2" library="rhoban" deviceset="OPEN-BLDC_IR2101" device="">
-<attribute name="FARNELL" value="8638730"/>
+<attribute name="FARNELL" value="8638756"/>
 </part>
 <part name="C2" library="SparkFun-Capacitors" deviceset="0.33UF/330NF" device="-0805-50V-10%" value="1µF">
-<attribute name="FARNELL" value="2528772"/>
+<attribute name="FARNELL" value="2496946"/>
 </part>
 <part name="DRV3" library="rhoban" deviceset="OPEN-BLDC_IR2101" device="">
-<attribute name="FARNELL" value="8638730"/>
+<attribute name="FARNELL" value="8638756"/>
 </part>
 <part name="C3" library="SparkFun-Capacitors" deviceset="0.33UF/330NF" device="-0805-50V-10%" value="1µF">
-<attribute name="FARNELL" value="2528772"/>
+<attribute name="FARNELL" value="2496946"/>
 </part>
 <part name="R1" library="SparkFun-Resistors" deviceset="RESISTOR" device="0805" value="10">
-<attribute name="FARNELL" value="2446904"/>
+<attribute name="FARNELL" value="2498048"/>
 </part>
 <part name="R2" library="SparkFun-Resistors" deviceset="RESISTOR" device="0805" value="10">
-<attribute name="FARNELL" value="2446904"/>
+<attribute name="FARNELL" value="2498048"/>
 </part>
 <part name="R3" library="SparkFun-Resistors" deviceset="RESISTOR" device="0805" value="10">
-<attribute name="FARNELL" value="2446904"/>
+<attribute name="FARNELL" value="2498048"/>
 </part>
 <part name="R4" library="SparkFun-Resistors" deviceset="RESISTOR" device="0805" value="10">
-<attribute name="FARNELL" value="2446904"/>
+<attribute name="FARNELL" value="2498048"/>
 </part>
 <part name="R5" library="SparkFun-Resistors" deviceset="RESISTOR" device="0805" value="10">
-<attribute name="FARNELL" value="2446904"/>
+<attribute name="FARNELL" value="2498048"/>
 </part>
 <part name="R6" library="SparkFun-Resistors" deviceset="RESISTOR" device="0805" value="10">
-<attribute name="FARNELL" value="2446904"/>
+<attribute name="FARNELL" value="2498048"/>
 </part>
 <part name="Q1" library="transistor-power" deviceset="BUK7Y12-40E" device="">
@@
 </part>
 <part name="C4" library="SparkFun-Passives" deviceset="CAP" device="0805" value="1000pF">
-<attribute name="FARNELL" value="2496935"/>
+<attribute name="FARNELL" value="2392334"/>
 </part>
 <part name="R20" library="SparkFun-Resistors" deviceset="RESISTOR" device="0805" value="2K">
@@
 </part>
 <part name="D5" library="SparkFun-DiscreteSemi" deviceset="DIODE" device="SOD" value="Schottky">
-<attribute name="FARNELL" value="2760406"/>
+<attribute name="FARNELL" value="8734593"/>
 </part>
 <part name="JP1" library="SparkFun-Jumpers" deviceset="JUMPER-SMT_2_NC_PASTE" device="_NO-SILK">
@@
 <part name="AGND20" library="supply1" deviceset="AGND" device=""/>
 <part name="C9" library="SparkFun-Passives" deviceset="CAP" device="0805" value="100nF">
-<attribute name="FARNELL" value="2496935"/>
+<attribute name="FARNELL" value="1759143RL"/>
 </part>
 <part name="C11" library="SparkFun-Passives" deviceset="CAP" device="0805" value="1uF">
-<attribute name="FARNELL" value="2496935"/>
+<attribute name="FARNELL" value="2496946"/>
 </part>
 <part name="C13" library="SparkFun-Passives" deviceset="CAP" device="0805" value="100nF">
-<attribute name="FARNELL" value="2496935"/>
+<attribute name="FARNELL" value="1759143RL"/>
 </part>
 <part name="3.3/4.5D3" library="supply1" deviceset="+3V3" device=""/>
 <part name="D6" library="SparkFun-DiscreteSemi" deviceset="DIODE" device="SOD" value="Schottky">
-<attribute name="FARNELL" value="2760406"/>
+<attribute name="FARNELL" value="8734593"/>
 </part>
 <part name="D1" library="SparkFun-DiscreteSemi" deviceset="DIODE" device="SOD" value="Signal">
@@
 </part>
 <part name="D2" library="SparkFun-DiscreteSemi" deviceset="DIODE" device="SOD" value="Schottky">
-<attribute name="FARNELL" value="2760406"/>
+<attribute name="FARNELL" value="8734593"/>
 </part>
 <part name="D7" library="SparkFun-DiscreteSemi" deviceset="DIODE" device="SOD" value="Signal">
@@
 </part>
 <part name="D3" library="SparkFun-DiscreteSemi" deviceset="DIODE" device="SOD" value="Schottky">
-<attribute name="FARNELL" value="2760406"/>
+<attribute name="FARNELL" value="8734593"/>
 </part>
 <part name="D10" library="SparkFun-DiscreteSemi" deviceset="DIODE" device="SOD" value="Signal">
@@
 </part>
 <part name="D12" library="SparkFun-DiscreteSemi" deviceset="DIODE" device="SOD" value="Schottky">
-<attribute name="FARNELL" value="2760406"/>
+<attribute name="FARNELL" value="8734593"/>
 </part>
 <part name="R7" library="SparkFun-Resistors" deviceset="RESISTOR" device="0805" value="10">
-<attribute name="FARNELL" value="2446904"/>
+<attribute name="FARNELL" value="2498048"/>
 <attribute name="PROD_ID" value=" "/>
 <attribute name="VALUE" value=" "/>
 </part>
 <part name="R8" library="SparkFun-Resistors" deviceset="RESISTOR" device="0805" value="10">
-<attribute name="FARNELL" value="2446904"/>
+<attribute name="FARNELL" value="2498048"/>
 <attribute name="PROD_ID" value=" "/>
 <attribute name="VALUE" value=" "/>
 </part>
 <part name="R9" library="SparkFun-Resistors" deviceset="RESISTOR" device="0805" value="10">
-<attribute name="FARNELL" value="2446904"/>
+<attribute name="FARNELL" value="2498048"/>
 <attribute name="PROD_ID" value=" "/>
 <attribute name="VALUE" value=" "/>
 </part>
 <part name="R10" library="SparkFun-Resistors" deviceset="RESISTOR" device="0805" value="10">
-<attribute name="FARNELL" value="2446904"/>
+<attribute name="FARNELL" value="2498048"/>
 <attribute name="PROD_ID" value=" "/>
 <attribute name="VALUE" value=" "/>
 </part>
 <part name="R11" library="SparkFun-Resistors" deviceset="RESISTOR" device="0805" value="10">
-<attribute name="FARNELL" value="2446904"/>
+<attribute name="FARNELL" value="2498048"/>
 <attribute name="PROD_ID" value=" "/>
 <attribute name="VALUE" value=" "/>
 </part>
 <part name="R12" library="SparkFun-Resistors" deviceset="RESISTOR" device="0805" value="10">
-<attribute name="FARNELL" value="2446904"/>
-<attribute name="PROD_ID" value=" "/>
-<attribute name="VALUE" value=" "/>
+<attribute name="FARNELL" value="2498048"/>
+<attribute name="PROD_ID" value=" "/>
+<attribute name="VALUE" value=" "/>
