File: brushless/rev2/brushless.brd (EAGLE design)
At the start: 30 x 48 mm, 72 parts, among them Q1 BUK7Y12-40E, Q2 BUK7Y12-40E, Q3 BUK7Y12-40E, Q4 BUK7Y12-40E, Q5 BUK7Y12-40E, Q6 BUK7Y12-40E, X2 MOTOR

Commit message: Passive values
Parts:
- C11: value 1000pF -> 1uF
- C13: value 1000pF -> 100nF
Changed lines of the file:
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@@
 <attribute name="VALUE" x="23.947" y="29.346" size="0.4064" layer="27" rot="R90"/>
 </element>
-<element name="C11" library="SparkFun-Passives" package="0805@1" value="1000pF" x="2.925" y="9.282" smashed="yes" rot="MR270">
+<element name="C11" library="SparkFun-Passives" package="0805@1" value="1uF" x="2.925" y="9.282" smashed="yes" rot="MR270">
 <attribute name="FARNELL" value="2496935" x="2.925" y="9.282" size="1.778" layer="28" rot="MR270" display="off"/>
 <attribute name="NAME" x="3.2425" y="7.377" size="0.6096" layer="26" ratio="20" rot="MR270"/>
 <attribute name="VALUE" x="4.322" y="10.298" size="0.4064" layer="28" rot="MR270"/>
 </element>
-<element name="C13" library="SparkFun-Passives" package="0805@1" value="1000pF" x="9.521" y="8.538" smashed="yes" rot="R270">
+<element name="C13" library="SparkFun-Passives" package="0805@1" value="100nF" x="9.521" y="8.538" smashed="yes" rot="R270">
 <attribute name="FARNELL" value="2496935" x="9.521" y="8.538" size="1.778" layer="27" rot="R270" display="off"/>
 <attribute name="NAME" x="10.3465" y="9.3" size="0.6096" layer="25" ratio="20" rot="R270"/>

Commit message: Fixing rev2 board/sch consistency
Parts:
- C1, C2, C3: value 10µF -> 1µF
- C9: value 1000pF -> 100nF
Changed lines of the file:
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@@
 <grid distance="1.27" unitdist="mm" unit="mm" style="lines" multiple="1" display="yes" altdistance="0.01" altunitdist="mm" altunit="mm"/>
 <layers>
-<layer number="1" name="Top" color="4" fill="1" visible="no" active="yes"/>
+<layer number="1" name="Top" color="4" fill="1" visible="yes" active="yes"/>
 <layer number="2" name="Route2" color="11" fill="1" visible="no" active="yes"/>
 <layer number="3" name="Route3" color="4" fill="3" visible="no" active="no"/>
@@
 <layer number="14" name="Route14" color="1" fill="6" visible="no" active="no"/>
 <layer number="15" name="Route15" color="14" fill="1" visible="no" active="yes"/>
-<layer number="16" name="Bottom" color="1" fill="1" visible="yes" active="yes"/>
+<layer number="16" name="Bottom" color="1" fill="1" visible="no" active="yes"/>
 <layer number="17" name="Pads" color="2" fill="1" visible="yes" active="yes"/>
 <layer number="18" name="Vias" color="2" fill="1" visible="yes" active="yes"/>
 <layer number="19" name="Unrouted" color="6" fill="1" visible="yes" active="yes"/>
 <layer number="20" name="Dimension" color="15" fill="1" visible="yes" active="yes"/>
-<layer number="21" name="tPlace" color="7" fill="1" visible="no" active="yes"/>
-<layer number="22" name="bPlace" color="7" fill="1" visible="yes" active="yes"/>
-<layer number="23" name="tOrigins" color="15" fill="1" visible="no" active="yes"/>
-<layer number="24" name="bOrigins" color="15" fill="1" visible="yes" active="yes"/>
-<layer number="25" name="tNames" color="7" fill="1" visible="no" active="yes"/>
-<layer number="26" name="bNames" color="7" fill="1" visible="yes" active="yes"/>
-<layer number="27" name="tValues" color="7" fill="1" visible="no" active="yes"/>
-<layer number="28" name="bValues" color="7" fill="1" visible="yes" active="yes"/>
-<layer number="29" name="tStop" color="7" fill="3" visible="no" active="yes"/>
-<layer number="30" name="bStop" color="7" fill="6" visible="yes" active="yes"/>
-<layer number="31" name="tCream" color="7" fill="4" visible="no" active="yes"/>
-<layer number="32" name="bCream" color="7" fill="5" visible="yes" active="yes"/>
-<layer number="33" name="tFinish" color="6" fill="3" visible="no" active="yes"/>
-<layer number="34" name="bFinish" color="6" fill="6" visible="yes" active="yes"/>
-<layer number="35" name="tGlue" color="7" fill="4" visible="no" active="yes"/>
-<layer number="36" name="bGlue" color="7" fill="5" visible="yes" active="yes"/>
-<layer number="37" name="tTest" color="7" fill="1" visible="no" active="yes"/>
-<layer number="38" name="bTest" color="7" fill="1" visible="yes" active="yes"/>
-<layer number="39" name="tKeepout" color="4" fill="11" visible="no" active="yes"/>
-<layer number="40" name="bKeepout" color="1" fill="11" visible="yes" active="yes"/>
+<layer number="21" name="tPlace" color="7" fill="1" visible="yes" active="yes"/>
+<layer number="22" name="bPlace" color="7" fill="1" visible="no" active="yes"/>
+<layer number="23" name="tOrigins" color="15" fill="1" visible="yes" active="yes"/>
+<layer number="24" name="bOrigins" color="15" fill="1" visible="no" active="yes"/>
+<layer number="25" name="tNames" color="7" fill="1" visible="yes" active="yes"/>
+<layer number="26" name="bNames" color="7" fill="1" visible="no" active="yes"/>
+<layer number="27" name="tValues" color="7" fill="1" visible="yes" active="yes"/>
+<layer number="28" name="bValues" color="7" fill="1" visible="no" active="yes"/>
+<layer number="29" name="tStop" color="7" fill="3" visible="yes" active="yes"/>
+<layer number="30" name="bStop" color="7" fill="6" visible="no" active="yes"/>
+<layer number="31" name="tCream" color="7" fill="4" visible="yes" active="yes"/>
+<layer number="32" name="bCream" color="7" fill="5" visible="no" active="yes"/>
+<layer number="33" name="tFinish" color="6" fill="3" visible="yes" active="yes"/>
+<layer number="34" name="bFinish" color="6" fill="6" visible="no" active="yes"/>
+<layer number="35" name="tGlue" color="7" fill="4" visible="yes" active="yes"/>
+<layer number="36" name="bGlue" color="7" fill="5" visible="no" active="yes"/>
+<layer number="37" name="tTest" color="7" fill="1" visible="yes" active="yes"/>
+<layer number="38" name="bTest" color="7" fill="1" visible="no" active="yes"/>
+<layer number="39" name="tKeepout" color="4" fill="11" visible="yes" active="yes"/>
+<layer number="40" name="bKeepout" color="1" fill="11" visible="no" active="yes"/>
 <layer number="41" name="tRestrict" color="4" fill="10" visible="yes" active="yes"/>
-<layer number="42" name="bRestrict" color="1" fill="10" visible="yes" active="yes"/>
+<layer number="42" name="bRestrict" color="1" fill="10" visible="no" active="yes"/>
 <layer number="43" name="vRestrict" color="2" fill="10" visible="yes" active="yes"/>
 <layer number="44" name="Drills" color="7" fill="1" visible="yes" active="yes"/>
@@
 <layer number="49" name="Reference" color="7" fill="1" visible="yes" active="yes"/>
 <layer number="50" name="dxf" color="7" fill="1" visible="no" active="no"/>
-<layer number="51" name="tDocu" color="7" fill="1" visible="no" active="yes"/>
-<layer number="52" name="bDocu" color="7" fill="1" visible="yes" active="yes"/>
+<layer number="51" name="tDocu" color="7" fill="1" visible="yes" active="yes"/>
+<layer number="52" name="bDocu" color="7" fill="1" visible="no" active="yes"/>
 <layer number="53" name="tGND_GNDA" color="7" fill="9" visible="no" active="no"/>
 <layer number="54" name="bGND_GNDA" color="1" fill="9" visible="no" active="no"/>
@@
 <layer number="101" name="Patch_Top" color="12" fill="4" visible="yes" active="yes"/>
 <layer number="102" name="Vscore" color="7" fill="1" visible="yes" active="yes"/>
-<layer number="103" name="tMap" color="7" fill="1" visible="no" active="yes"/>
+<layer number="103" name="tMap" color="7" fill="1" visible="yes" active="yes"/>
 <layer number="104" name="Name" color="16" fill="1" visible="yes" active="yes"/>
 <layer number="105" name="tPlate" color="7" fill="1" visible="yes" active="yes"/>
-<layer number="106" name="bPlate" color="7" fill="1" visible="yes" active="yes"/>
+<layer number="106" name="bPlate" color="7" fill="1" visible="no" active="yes"/>
 <layer number="107" name="Crop" color="7" fill="1" visible="yes" active="yes"/>
 <layer number="108" name="tplace-old" color="10" fill="1" visible="yes" active="yes"/>
@@
 <layer number="110" name="fp0" color="7" fill="1" visible="yes" active="yes"/>
 <layer number="111" name="LPC17xx" color="7" fill="1" visible="yes" active="yes"/>
-<layer number="112" name="tSilk" color="7" fill="1" visible="no" active="yes"/>
+<layer number="112" name="tSilk" color="7" fill="1" visible="yes" active="yes"/>
 <layer number="113" name="IDFDebug" color="4" fill="1" visible="yes" active="yes"/>
 <layer number="114" name="Badge_Outline" color="7" fill="1" visible="yes" active="yes"/>
@@
 <layer number="119" name="KAP_TEKEN" color="7" fill="1" visible="yes" active="yes"/>
 <layer number="120" name="KAP_MAAT1" color="7" fill="1" visible="yes" active="yes"/>
-<layer number="121" name="_tsilk" color="7" fill="1" visible="no" active="yes"/>
+<layer number="121" name="_tsilk" color="7" fill="1" visible="yes" active="yes"/>
 <layer number="122" name="_bsilk" color="7" fill="1" visible="yes" active="yes"/>
 <layer number="123" name="tTestmark" color="7" fill="1" visible="yes" active="yes"/>
@@
 <attribute name="VALUE" x="19.9164" y="29.4628" size="0.6096" layer="27" font="vector" ratio="20" rot="R90"/>
 </element>
-<element name="C1" library="SparkFun-Capacitors" package="0805" value="10µF" x="6.3496" y="25.1198" smashed="yes" rot="MR90">
+<element name="C1" library="SparkFun-Capacitors" package="0805" value="1µF" x="6.3496" y="25.1198" smashed="yes" rot="MR90">
 <attribute name="PROD_ID" value="CAP-08469" x="6.3496" y="25.1198" size="1.778" layer="28" rot="MR90" display="off"/>
 <attribute name="VALUE" value="0.33µF" x="6.3496" y="25.1198" size="1.778" layer="28" rot="MR90" display="off"/>
@@
 <attribute name="NAME" x="8.7293" y="18.1752" size="0.8128" layer="26" ratio="10" rot="MR90"/>
 </element>
-<element name="C2" library="SparkFun-Capacitors" package="0805" value="10µF" x="13.592" y="27.2488" smashed="yes" rot="MR90">
+<element name="C2" library="SparkFun-Capacitors" package="0805" value="1µF" x="13.592" y="27.2488" smashed="yes" rot="MR90">
 <attribute name="PROD_ID" value="CAP-08469" x="12.322" y="27.2488" size="1.778" layer="28" rot="MR90" display="off"/>
 <attribute name="VALUE" value="0.33µF" x="12.322" y="27.2488" size="1.778" layer="28" rot="MR90" display="off"/>
@@
 <attribute name="NAME" x="16.0145" y="20.4072" size="0.8128" layer="26" ratio="10" rot="MR90"/>
 </element>
-<element name="C3" library="SparkFun-Capacitors" package="0805" value="10µF" x="20.7328" y="28.6394" smashed="yes" rot="MR90">
+<element name="C3" library="SparkFun-Capacitors" package="0805" value="1µF" x="20.7328" y="28.6394" smashed="yes" rot="MR90">
 <attribute name="PROD_ID" value="CAP-08469" x="19.4628" y="28.6394" size="1.778" layer="28" rot="MR90" display="off"/>
 <attribute name="VALUE" value="0.33µF" x="19.4628" y="28.6394" size="1.778" layer="28" rot="MR90" display="off"/>
@@
 <attribute name="VALUE" x="5.703" y="16.405" size="0.4064" layer="28" rot="MR90"/>
 </element>
-<element name="C9" library="SparkFun-Passives" package="0805@1" value="1000pF" x="22.55" y="30.362" smashed="yes" rot="R90">
+<element name="C9" library="SparkFun-Passives" package="0805@1" value="100nF" x="22.55" y="30.362" smashed="yes" rot="R90">
 <attribute name="FARNELL" value="2496935" x="22.55" y="30.362" size="1.778" layer="27" rot="R90" display="off"/>
 <attribute name="NAME" x="21.5975" y="29.6" size="0.6096" layer="25" ratio="20" rot="R90"/>

Commit message: Improving values indications
Parts:
- D1, D10, D11, D7, D8, D9: value (none) -> Signal
- D12, D2, D3, D5, D6: value (none) -> Schottky
Changed lines of the file:
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@@
 <attribute name="VALUE" x="28.541784375" y="38.381703125" size="1.27" layer="27" ratio="10" rot="R135"/>
 </element>
-<element name="D5" library="SparkFun-DiscreteSemi" package="SOD-323" value="" x="28.583" y="1.509" smashed="yes" rot="MR270">
-<attribute name="FARNELL" value="8737843RL" x="28.583" y="1.509" size="1.778" layer="28" rot="MR270" display="off"/>
+<element name="D5" library="SparkFun-DiscreteSemi" package="SOD-323" value="Schottky" x="28.583" y="1.509" smashed="yes" rot="MR270">
+<attribute name="FARNELL" value="2760406" x="28.583" y="1.509" size="1.778" layer="28" rot="MR270" display="off"/>
 <attribute name="NAME" x="27.44" y="1.89" size="0.6096" layer="26" ratio="20" rot="MR270"/>
 <attribute name="VALUE" x="29.98" y="2.525" size="0.4064" layer="28" rot="MR270"/>
@@
 <attribute name="VALUE" x="8.124" y="9.554" size="0.4064" layer="27" rot="R270"/>
 </element>
-<element name="D6" library="SparkFun-DiscreteSemi" package="SOD-323" value="" x="7.073" y="21.094" smashed="yes" rot="MR270">
-<attribute name="FARNELL" value="8737843RL" x="3.573" y="24.294" size="1.778" layer="28" rot="MR270" display="off"/>
+<element name="D6" library="SparkFun-DiscreteSemi" package="SOD-323" value="Schottky" x="7.073" y="21.094" smashed="yes" rot="MR270">
+<attribute name="FARNELL" value="2760406" x="3.573" y="24.294" size="1.778" layer="28" rot="MR270" display="off"/>
 <attribute name="NAME" x="8.47" y="21.602" size="0.6096" layer="26" ratio="20" rot="MR270"/>
 <attribute name="VALUE" x="8.47" y="22.11" size="0.4064" layer="28" rot="MR270"/>
 </element>
-<element name="D1" library="SparkFun-DiscreteSemi" package="SOD-323" value="" x="4.492" y="25.616" smashed="yes" rot="MR90">
-<attribute name="FARNELL" value="8737843RL" x="4.492" y="25.616" size="1.778" layer="28" rot="MR90" display="off"/>
+<element name="D1" library="SparkFun-DiscreteSemi" package="SOD-323" value="Signal" x="4.492" y="25.616" smashed="yes" rot="MR90">
+<attribute name="FARNELL" value="1843678RL" x="4.492" y="25.616" size="1.778" layer="28" rot="MR90" display="off"/>
 <attribute name="NAME" x="5.127" y="27.013" size="0.6096" layer="26" ratio="20" rot="MR90"/>
 <attribute name="VALUE" x="3.095" y="24.6" size="0.4064" layer="28" rot="MR90"/>
 </element>
-<element name="D2" library="SparkFun-DiscreteSemi" package="SOD-323" value="" x="14.527" y="21.045" smashed="yes" rot="MR270">
-<attribute name="FARNELL" value="8737843RL" x="14.527" y="21.045" size="1.778" layer="28" rot="MR270" display="off"/>
+<element name="D2" library="SparkFun-DiscreteSemi" package="SOD-323" value="Schottky" x="14.527" y="21.045" smashed="yes" rot="MR270">
+<attribute name="FARNELL" value="2760406" x="14.527" y="21.045" size="1.778" layer="28" rot="MR270" display="off"/>
 <attribute name="NAME" x="16.051" y="21.807" size="0.6096" layer="26" ratio="20" rot="MR270"/>
 <attribute name="VALUE" x="15.924" y="22.061" size="0.4064" layer="28" rot="MR270"/>
 </element>
-<element name="D7" library="SparkFun-DiscreteSemi" package="SOD-323" value="" x="11.737" y="25.735" smashed="yes" rot="MR90">
-<attribute name="FARNELL" value="8737843RL" x="11.737" y="25.735" size="1.778" layer="28" rot="MR90" display="off"/>
+<element name="D7" library="SparkFun-DiscreteSemi" package="SOD-323" value="Signal" x="11.737" y="25.735" smashed="yes" rot="MR90">
+<attribute name="FARNELL" value="1843678RL" x="11.737" y="25.735" size="1.778" layer="28" rot="MR90" display="off"/>
 <attribute name="NAME" x="12.626" y="23.703" size="0.6096" layer="26" ratio="20" rot="MR90"/>
 <attribute name="VALUE" x="10.34" y="24.719" size="0.4064" layer="28" rot="MR90"/>
 </element>
-<element name="D8" library="SparkFun-DiscreteSemi" package="SOD-323" value="" x="12.355" y="25.999" smashed="yes" rot="R90">
-<attribute name="FARNELL" value="8737843RL" x="12.355" y="25.999" size="1.778" layer="27" rot="R90" display="off"/>
+<element name="D8" library="SparkFun-DiscreteSemi" package="SOD-323" value="Signal" x="12.355" y="25.999" smashed="yes" rot="R90">
+<attribute name="FARNELL" value="1843678RL" x="12.355" y="25.999" size="1.778" layer="27" rot="R90" display="off"/>
 <attribute name="NAME" x="13.752" y="25.745" size="0.6096" layer="25" ratio="20" rot="R90"/>
 <attribute name="VALUE" x="13.752" y="24.983" size="0.4064" layer="27" rot="R90"/>
 </element>
-<element name="D9" library="SparkFun-DiscreteSemi" package="SOD-323" value="" x="4.931" y="25.567" smashed="yes" rot="R90">
-<attribute name="FARNELL" value="8737843RL" x="4.931" y="25.567" size="1.778" layer="27" rot="R90" display="off"/>
+<element name="D9" library="SparkFun-DiscreteSemi" package="SOD-323" value="Signal" x="4.931" y="25.567" smashed="yes" rot="R90">
+<attribute name="FARNELL" value="1843678RL" x="4.931" y="25.567" size="1.778" layer="27" rot="R90" display="off"/>
 <attribute name="NAME" x="6.455" y="24.805" size="0.6096" layer="25" ratio="20" rot="R90"/>
 <attribute name="VALUE" x="6.328" y="24.551" size="0.4064" layer="27" rot="R90"/>
 </element>
-<element name="D3" library="SparkFun-DiscreteSemi" package="SOD-323" value="" x="25.537" y="22.061" smashed="yes" rot="MR270">
-<attribute name="FARNELL" value="8737843RL" x="25.537" y="22.061" size="1.778" layer="28" rot="MR270" display="off"/>
+<element name="D3" library="SparkFun-DiscreteSemi" package="SOD-323" value="Schottky" x="25.537" y="22.061" smashed="yes" rot="MR270">
+<attribute name="FARNELL" value="2760406" x="25.537" y="22.061" size="1.778" layer="28" rot="MR270" display="off"/>
 <attribute name="NAME" x="24.521" y="22.95" size="0.6096" layer="26" ratio="20" rot="MR270"/>
 <attribute name="VALUE" x="26.934" y="23.077" size="0.4064" layer="28" rot="MR270"/>
 </element>
-<element name="D10" library="SparkFun-DiscreteSemi" package="SOD-323" value="" x="16.206" y="28.731" smashed="yes" rot="MR90">
-<attribute name="FARNELL" value="8737843RL" x="16.206" y="28.731" size="1.778" layer="28" rot="MR90" display="off"/>
+<element name="D10" library="SparkFun-DiscreteSemi" package="SOD-323" value="Signal" x="16.206" y="28.731" smashed="yes" rot="MR90">
+<attribute name="FARNELL" value="1843678RL" x="16.206" y="28.731" size="1.778" layer="28" rot="MR90" display="off"/>
 <attribute name="NAME" x="17.222" y="27.842" size="0.6096" layer="26" ratio="20" rot="MR90"/>
 <attribute name="VALUE" x="14.809" y="27.715" size="0.4064" layer="28" rot="MR90"/>
 </element>
-<element name="D11" library="SparkFun-DiscreteSemi" package="SOD-323" value="" x="17.166" y="29.428" smashed="yes" rot="R90">
-<attribute name="FARNELL" value="8737843RL" x="17.166" y="29.428" size="1.778" layer="27" rot="R90" display="off"/>
+<element name="D11" library="SparkFun-DiscreteSemi" package="SOD-323" value="Signal" x="17.166" y="29.428" smashed="yes" rot="R90">
+<attribute name="FARNELL" value="1843678RL" x="17.166" y="29.428" size="1.778" layer="27" rot="R90" display="off"/>
 <attribute name="NAME" x="16.15" y="28.539" size="0.6096" layer="25" ratio="20" rot="R90"/>
 <attribute name="VALUE" x="18.563" y="28.412" size="0.4064" layer="27" rot="R90"/>
 </element>
-<element name="D12" library="SparkFun-DiscreteSemi" package="SOD-323" value="" x="28.742" y="2.044" smashed="yes" rot="R270">
-<attribute name="FARNELL" value="8737843RL" x="32.242" y="5.244" size="1.778" layer="27" rot="R270" display="off"/>
+<element name="D12" library="SparkFun-DiscreteSemi" package="SOD-323" value="Schottky" x="28.742" y="2.044" smashed="yes" rot="R270">
+<attribute name="FARNELL" value="2760406" x="32.242" y="5.244" size="1.778" layer="27" rot="R270" display="off"/>
 <attribute name="NAME" x="28.869" y="5.6" size="0.6096" layer="25" ratio="20" rot="R270"/>
 <attribute name="VALUE" x="27.345" y="3.06" size="0.4064" layer="27" rot="R270"/>
