File: brushless/brushless.brd (EAGLE design)
At the start: 30 x 48 mm, 72 parts, among them Q1 BUK7Y12-40E, Q2 BUK7Y12-40E, Q3 BUK7Y12-40E, Q4 BUK7Y12-40E, Q5 BUK7Y12-40E, Q6 BUK7Y12-40E, X2 MOTOR

Commit message: Values
Parts:
- C1, C2, C3: value 10µF -> 1µF
Changed lines of the file:
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@@
 <attribute name="VALUE" x="19.9164" y="29.4628" size="0.6096" layer="27" font="vector" ratio="20" rot="R90"/>
 </element>
-<element name="C1" library="SparkFun-Capacitors" package="0805" value="10µF" x="6.3496" y="25.1198" smashed="yes" rot="MR90">
+<element name="C1" library="SparkFun-Capacitors" package="0805" value="1µF" x="6.3496" y="25.1198" smashed="yes" rot="MR90">
 <attribute name="PROD_ID" value="CAP-08469" x="6.3496" y="25.1198" size="1.778" layer="28" rot="MR90" display="off"/>
 <attribute name="VALUE" value="0.33µF" x="6.3496" y="25.1198" size="1.778" layer="28" rot="MR90" display="off"/>
@@
 <attribute name="NAME" x="8.7293" y="18.1752" size="0.8128" layer="26" ratio="10" rot="MR90"/>
 </element>
-<element name="C2" library="SparkFun-Capacitors" package="0805" value="10µF" x="13.592" y="27.2488" smashed="yes" rot="MR90">
+<element name="C2" library="SparkFun-Capacitors" package="0805" value="1µF" x="13.592" y="27.2488" smashed="yes" rot="MR90">
 <attribute name="PROD_ID" value="CAP-08469" x="12.322" y="27.2488" size="1.778" layer="28" rot="MR90" display="off"/>
 <attribute name="VALUE" value="0.33µF" x="12.322" y="27.2488" size="1.778" layer="28" rot="MR90" display="off"/>
@@
 <attribute name="NAME" x="16.0145" y="20.4072" size="0.8128" layer="26" ratio="10" rot="MR90"/>
 </element>
-<element name="C3" library="SparkFun-Capacitors" package="0805" value="10µF" x="20.7328" y="28.6394" smashed="yes" rot="MR90">
+<element name="C3" library="SparkFun-Capacitors" package="0805" value="1µF" x="20.7328" y="28.6394" smashed="yes" rot="MR90">
 <attribute name="PROD_ID" value="CAP-08469" x="19.4628" y="28.6394" size="1.778" layer="28" rot="MR90" display="off"/>
 <attribute name="VALUE" value="0.33µF" x="19.4628" y="28.6394" size="1.778" layer="28" rot="MR90" display="off"/>

Commit message: Passive values
Parts:
- C11: value 1000pF -> 1uF
- C13: value 1000pF -> 100nF
Changed lines of the file:
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@@
 <attribute name="VALUE" x="23.947" y="29.346" size="0.4064" layer="27" rot="R90"/>
 </element>
-<element name="C11" library="SparkFun-Passives" package="0805@1" value="1000pF" x="2.925" y="9.282" smashed="yes" rot="MR270">
+<element name="C11" library="SparkFun-Passives" package="0805@1" value="1uF" x="2.925" y="9.282" smashed="yes" rot="MR270">
 <attribute name="FARNELL" value="2496935" x="2.925" y="9.282" size="1.778" layer="28" rot="MR270" display="off"/>
 <attribute name="NAME" x="3.2425" y="7.377" size="0.6096" layer="26" ratio="20" rot="MR270"/>
 <attribute name="VALUE" x="4.322" y="10.298" size="0.4064" layer="28" rot="MR270"/>
 </element>
-<element name="C13" library="SparkFun-Passives" package="0805@1" value="1000pF" x="9.521" y="8.538" smashed="yes" rot="R270">
+<element name="C13" library="SparkFun-Passives" package="0805@1" value="100nF" x="9.521" y="8.538" smashed="yes" rot="R270">
 <attribute name="FARNELL" value="2496935" x="9.521" y="8.538" size="1.778" layer="27" rot="R270" display="off"/>
 <attribute name="NAME" x="10.3465" y="9.3" size="0.6096" layer="25" ratio="20" rot="R270"/>

Commit message: Improving values indications
Parts:
- C9: value 1000pF -> 100nF
- D1, D10, D11, D7, D8, D9: value (none) -> Signal
- D12, D2, D3, D5, D6: value (none) -> Schottky
