File: mainboard/backup/mainboard.brd (EAGLE design)
At the start: 158.8 x 136.4 mm, 69 parts, among them T2 NPN_BC817,215, U1 CD4051BM, X2 JST-XH-07-PIN-LONG-PAD

Commit message: mainboard rerouted
Parts:
- moved R10 60.7 mm to (-11.5, 22.0), turned to 180 degrees
- moved U1 57.6 mm to (-7.55, 12.0)
- moved C10 56.8 mm to (0.33, 9.94)
- moved R11 55.5 mm to (-11.3, 18.7)
- moved DRIVER2 53.4 mm to (31.4, -48.0), turned to 0 degrees
- moved DRIVER1 53.0 mm to (61.5, 51.9), turned to 180 degrees
- moved DRIVER4 52.5 mm to (-24.3, 45.6), turned to 180 degrees
- moved DRIVER5 52.5 mm to (7.52, 29.3), turned to 180 degrees
- moved DRIVER3 52.1 mm to (-54.1, -48.1), turned to 0 degrees
- moved D4 47.8 mm to (-9.86, 30.2)
- moved D5 45.2 mm to (46.4, 47.9), turned to 270 degrees
- moved C7 44.7 mm to (-18.1, -21.2), turned to 180 degrees
- moved C11 42.0 mm to (24.2, -44.6), flipped to the top, turned to 180 degrees
- moved D1 39.9 mm to (46.6, -40.2), turned to 90 degrees
- moved D3 38.0 mm to (-39.5, 41.9), turned to 270 degrees
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Routing:
- net +3V3: track 617.4 -> 99.8 mm, vias 7 -> 0
- net V+: track 163.8 -> 395.9 mm
- net DRIVERS_SCK: track 155.2 -> 383.2 mm, vias 4 -> 1
- net DRIVERS_MOSI: track 152.6 -> 374.8 mm, vias 4 -> 5
- net DRIVERS_MISO: track 158.3 -> 376.4 mm
- net BUZZER: track 207.8 -> 0.00 mm, vias 1 -> 0
- net VCC: track 223.4 -> 57.1 mm, vias 3 -> 0
- net COM_CE1: track 132.7 -> 0.00 mm, vias 1 -> 0
- net COM_CE3: track 119.2 -> 0.00 mm, vias 1 -> 0
- net ADDR1: track 117.5 -> 0.00 mm, vias 2 -> 0
- net CS_COM_3: track 113.3 -> 0.00 mm
- net CS_COM_2: track 110.9 -> 0.00 mm, vias 3 -> 0
- net IRQ2: track 103.1 -> 0.00 mm, vias 1 -> 0
- net IRQ1: track 102.2 -> 0.00 mm, vias 1 -> 0
- net IRQ3: track 98.2 -> 3.95 mm, vias 1 -> 0
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- removed copper zone on layer 1, net GND
- removed copper zone on layer 15, net GND
- removed copper zone on layer 16, net GND
- removed copper zone on layer 1, net N$4
