File: mainboard/backup/mainboard_v2.brd (EAGLE design)
At the start: 158.8 x 136.4 mm, 69 parts, among them T2 NPN_BC817,215, U1 CD4051BM, X2 JST-XH-07-PIN-LONG-PAD

Commit message: mainboard rerouted
Parts:
- moved D5 45.2 mm to (46.4, 47.9), turned to 270 degrees
- moved C7 44.7 mm to (-18.1, -21.2), turned to 180 degrees
- moved D1 39.9 mm to (46.6, -40.2), turned to 90 degrees
- moved C11 23.1 mm to (-3.51, -25.8), flipped to the top, turned to 180 degrees
- moved C1 19.0 mm to (-1.52, -49.5), flipped to the top, turned to 180 degrees
- moved U$3 17.7 mm to (-13.7, -25.8), turned to 180 degrees
- moved U$6 15.0 mm to (-10.4, -44.1)
- moved R8 14.9 mm to (-15.2, -57.8), turned to 90 degrees
- moved REG3.3V1 14.2 mm to (-22.6, -37.2)
- moved REG3.3V 13.5 mm to (-22.7, -23.5)
- moved REG5V 13.3 mm to (2.27, -33.1), turned to 90 degrees
- moved U$4 12.8 mm to (-0.47, -41.6)
- moved D4 12.8 mm to (3.60, -14.5)
- moved D3 11.8 mm to (-37.6, 6.52), turned to 0 degrees
- moved C2 9.63 mm to (-19.0, -39.8), flipped to the top, turned to 180 degrees
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Routing:
- net +3V3: track 617.4 -> 39.1 mm, vias 7 -> 0
- net +12V: track 239.1 -> 0.00 mm, vias 5 -> 0
- net VCC: track 223.4 -> 0.00 mm, vias 3 -> 0
- net V+: track 163.8 -> 7.62 mm
- net GND: track 187.9 -> 38.3 mm, vias 35 -> 0
- net COM_CE3: track 119.2 -> 0.00 mm, vias 1 -> 0
- net CS_COM_3: track 113.3 -> 0.00 mm
- net IRQ3: track 98.2 -> 0.00 mm, vias 1 -> 0
- net KICK1: track 92.0 -> 0.00 mm, vias 2 -> 0
- net ADDR3: track 86.5 -> 0.00 mm, vias 2 -> 0
- net KICK2: track 81.9 -> 0.00 mm
- net MUX: track 81.8 -> 0.00 mm
- net BOOST_EN: track 81.7 -> 0.00 mm
- net ADDR2: track 62.7 -> 0.00 mm, vias 2 -> 0
- net HALL4: track 61.8 -> 2.64 mm, vias 1 -> 0
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- removed copper zone on layer 1, net GND
- removed copper zone on layer 15, net GND
- removed copper zone on layer 16, net GND
- removed copper zone on layer 1, net N$4
